File: PCB Files/Circuit-Teensy32-Full-Board/OpeNITHM-full.kicad_pcb (KiCad board)
At the start: 2 copper layers, 480 x 160 mm, 109 parts, among them J3 Conn_02x07_Odd_Even, J4 Conn_02x03_Odd_Even, J5 Conn_02x04_Odd_Even, U1 Teensy-LC, U2 74HC4051D, U3 74HC4051D, U4 74HC4051D, U5 74HC4051D

Commit message: Preliminary upload of the Fullboard v2.0 PCB, and it's separate LED board. Nothing here should be purchased, this is just uploaded for reviewing.
Parts:
- removed H17, H18: MountingHole, MountingHole:MountingHole_3.2mm_M3_ISO14580
- removed JP1: SolderJumper_3_Open, Jumper:SolderJumper-3_P1.3mm_Open_RoundedPad1.0x1.5mm_NumberLabels
- removed R17, R18, R19: 33, Resistor_THT:R_Axial_DIN0207_L6.3mm_D2.5mm_P7.62mm_Horizontal
- removed R20, R21, R22, R23, R24, R25: R_AIR, Resistor_THT:R_Axial_DIN0204_L3.6mm_D1.6mm_P5.08mm_Horizontal
- added C36: 100nF, Capacitor_SMD:C_0603_1608Metric, F.Cu at (223.4, 124.0)
- added C37: 100nF, Capacitor_SMD:C_0603_1608Metric, F.Cu at (232.7, 124.0)
- added C38: 100nF, Capacitor_SMD:C_0603_1608Metric, F.Cu at (242.1, 124.0)
- added C39: 100nF, Capacitor_SMD:C_0603_1608Metric, F.Cu at (251.4, 124.0)
- added C40: 100nF, Capacitor_SMD:C_0603_1608Metric, F.Cu at (260.7, 124.0)
- added C41: 100nF, Capacitor_SMD:C_0603_1608Metric, F.Cu at (270.1, 124.0)
- added C42: 100nF, Capacitor_SMD:C_0603_1608Metric, F.Cu at (279.4, 124.0)
- added C43: 100nF, Capacitor_SMD:C_0603_1608Metric, F.Cu at (288.7, 124.0)
- added C44: 100nF, Capacitor_SMD:C_0603_1608Metric, F.Cu at (298.1, 124.0)
- added C45: 100nF, Capacitor_SMD:C_0603_1608Metric, F.Cu at (307.4, 124.0)
- added C46: 100nF, Capacitor_SMD:C_0603_1608Metric, F.Cu at (316.7, 124.0)
- added C47: 100nF, Capacitor_SMD:C_0603_1608Metric, F.Cu at (326.1, 124.0)
- added C48: 100nF, Capacitor_SMD:C_0603_1608Metric, F.Cu at (335.4, 124.0)
- added C49: 100nF, Capacitor_SMD:C_0603_1608Metric, F.Cu at (344.7, 124.0)
- added C50: 100nF, Capacitor_SMD:C_0603_1608Metric, F.Cu at (354.1, 124.0)
- added C51: 100nF, Capacitor_SMD:C_0603_1608Metric, F.Cu at (363.4, 124.0)
- added D32: SK6812_SIDE-A, LED_SMD:LED_SK6812_SIDE-A_4020_4.0mmX2.0mm, F.Cu at (222.7, 120.0)
- added D33: SK6812_SIDE-A, LED_SMD:LED_SK6812_SIDE-A_4020_4.0mmX2.0mm, F.Cu at (232.0, 120.0)
- added D34: SK6812_SIDE-A, LED_SMD:LED_SK6812_SIDE-A_4020_4.0mmX2.0mm, F.Cu at (241.3, 120.0)
- added D35: SK6812_SIDE-A, LED_SMD:LED_SK6812_SIDE-A_4020_4.0mmX2.0mm, F.Cu at (250.7, 120.0)
- added D36: SK6812_SIDE-A, LED_SMD:LED_SK6812_SIDE-A_4020_4.0mmX2.0mm, F.Cu at (260.0, 120.0)
- added D37: SK6812_SIDE-A, LED_SMD:LED_SK6812_SIDE-A_4020_4.0mmX2.0mm, F.Cu at (269.3, 120.0)
- added D38: SK6812_SIDE-A, LED_SMD:LED_SK6812_SIDE-A_4020_4.0mmX2.0mm, F.Cu at (278.7, 120.0)
- added D39: SK6812_SIDE-A, LED_SMD:LED_SK6812_SIDE-A_4020_4.0mmX2.0mm, F.Cu at (288.0, 120.0)
- added D40: SK6812_SIDE-A, LED_SMD:LED_SK6812_SIDE-A_4020_4.0mmX2.0mm, F.Cu at (297.3, 120.0)
- added D41: SK6812_SIDE-A, LED_SMD:LED_SK6812_SIDE-A_4020_4.0mmX2.0mm, F.Cu at (306.7, 120.0)
- added D42: SK6812_SIDE-A, LED_SMD:LED_SK6812_SIDE-A_4020_4.0mmX2.0mm, F.Cu at (316.0, 120.0)
- added D43: SK6812_SIDE-A, LED_SMD:LED_SK6812_SIDE-A_4020_4.0mmX2.0mm, F.Cu at (325.3, 120.0)
- added D44: SK6812_SIDE-A, LED_SMD:LED_SK6812_SIDE-A_4020_4.0mmX2.0mm, F.Cu at (334.7, 120.0)
- added D45: SK6812_SIDE-A, LED_SMD:LED_SK6812_SIDE-A_4020_4.0mmX2.0mm, F.Cu at (344.0, 120.0)
- added D46: SK6812_SIDE-A, LED_SMD:LED_SK6812_SIDE-A_4020_4.0mmX2.0mm, F.Cu at (353.3, 120.0)
- added D47: SK6812_SIDE-A, LED_SMD:LED_SK6812_SIDE-A_4020_4.0mmX2.0mm, F.Cu at (362.7, 120.0)
- added D48: D_Schottky, Diode_SMD:D_SMA, F.Cu at (140.3, 10.9)
- added D49: D_Schottky, Diode_SMD:D_SMA, F.Cu at (124.5, 10.9)
- added J1: USB_C_Receptacle, Connector_USB:USB_C_Receptacle_GCT_USB4085, B.Cu at (145.0, 11.1)
- added J10: Conn_01x03, Connector_PinHeader_2.54mm:PinHeader_1x03_P2.54mm_Vertical, F.Cu at (375.2, 123.7)
- added J2: Conn_01x09, Connector_JST:JST_PH_S9B-PH-K_1x09_P2.00mm_Horizontal, B.Cu at (-85.5, 146.0)
- added J6: Conn_01x04, Connector_JST:JST_PH_S4B-PH-K_1x04_P2.00mm_Horizontal, B.Cu at (-85.5, 124.5)
- added J7: Barrel_Jack, Connector_BarrelJack:BarrelJack_Horizontal, B.Cu at (131.4, 16.2)
- added J8: Conn_01x02, Connector_PinHeader_2.54mm:PinHeader_1x02_P2.54mm_Vertical, B.Cu at (128.0, 139.7)
- added J9: Conn_01x03, Connector_PinHeader_2.54mm:PinHeader_1x03_P2.54mm_Vertical, F.Cu at (-74.2, 123.7)
- added LOGO3: Logo, OpeNITHM:openithm-logo, F.Cu at (352.0, 138.0)
- added R5: 5.1k, Resistor_SMD:R_0603_1608Metric, F.Cu at (150.3, 15.0)
- added R6: 5.1k, Resistor_SMD:R_0603_1608Metric, F.Cu at (150.3, 17.0)
- added TP1: +5V, TestPoint:TestPoint_Pad_D1.5mm, B.Cu at (158.5, 9.00)
- added TP2: D-, TestPoint:TestPoint_Pad_D1.5mm, B.Cu at (161.5, 9.00)
- added TP3: D+, TestPoint:TestPoint_Pad_D1.5mm, B.Cu at (164.5, 9.00)
- added TP4: GND, TestPoint:TestPoint_Pad_D1.5mm, B.Cu at (167.5, 9.00)
- D1, D10, D11, D12, D13, D14, D15, D16, D17, D18, D19, D2, D20, D21, D22, D23, D24, D25, D26, D27, D28, D29, D3, D30, D31, D4, D5, D6, D7, D8, D9: value WS2812B-B -> SK6812_SIDE-A; footprint LED_SMD:LED_WS2812B_PLCC4_5.0x5.0mm_P3.2mm -> LED_SMD:LED_SK6812_SIDE-A_4020_4.0mmX2.0mm
- J3: value Conn_02x07_Odd_Even -> Conn_01x09; footprint Connector_PinHeader_2.54mm:PinHeader_2x07_P2.54mm_Horizontal -> Connector_JST:JST_PH_S9B-PH-K_1x09_P2.00mm_Horizontal
- J4: value Conn_02x03_Odd_Even -> Conn_02x05_Odd_Even; footprint Connector_PinHeader_2.54mm:PinHeader_2x03_P2.54mm_Horizontal -> Connector_PinHeader_2.54mm:PinHeader_2x05_P2.54mm_Horizontal
- J5: value Conn_02x04_Odd_Even -> Conn_01x04; footprint Connector_PinHeader_2.54mm:PinHeader_2x04_P2.54mm_Horizontal -> Connector_JST:JST_PH_S4B-PH-K_1x04_P2.00mm_Horizontal
- LOGO1: moved to F.Cu
- LOGO2: footprint OpeNITHM:openithm-logo -> OpeNITHM:openithm-big; moved to B.Cu
- moved J4 479.8 mm to (378.5, 20.6), turned to 90 degrees
- moved U1 223.0 mm to (149.9, 141.0)
- moved H15 169.1 mm to (178.0, 132.0)
- moved C35 156.1 mm to (214.1, 124.0)
- moved D31 156.1 mm to (213.3, 120.0)
- moved C34 150.7 mm to (204.7, 124.0)
- moved D30 150.7 mm to (204.0, 120.0)
- moved C33 145.3 mm to (195.4, 124.0)
- moved D29 145.3 mm to (194.7, 120.0)
- moved C32 139.9 mm to (186.1, 124.0)
- moved D28 139.8 mm to (185.3, 120.0)
- moved C31 134.5 mm to (176.7, 124.0)
- moved D27 134.4 mm to (176.0, 120.0)
- moved C30 129.1 mm to (167.4, 124.0)
- moved D26 129.0 mm to (166.7, 120.0)
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Connections:
- D1 pad 1: +5V -> /RGB_DO_BUF
- D1 pad 2: Net-(D1-Pad2) -> +5V
- D1 pad 3: GND -> Net-(D1-Pad3)
- D1 pad 4: /RGB_DO_BUF -> GND
- D10 pad 1: +5V -> Net-(D10-Pad1)
- D10 pad 2: Net-(D10-Pad2) -> +5V
- D10 pad 3: GND -> Net-(D10-Pad3)
- D10 pad 4: Net-(D10-Pad4) -> GND
- D11 pad 1: +5V -> Net-(D10-Pad1)
- D11 pad 2: Net-(D11-Pad2) -> +5V
- D11 pad 3: GND -> Net-(D11-Pad3)
- D11 pad 4: Net-(D10-Pad2) -> GND
- D12 pad 1: +5V -> Net-(D11-Pad3)
- D12 pad 2: Net-(D12-Pad2) -> +5V
- D12 pad 3: GND -> Net-(D12-Pad3)
- D12 pad 4: Net-(D11-Pad2) -> GND
- D13 pad 1: +5V -> Net-(D12-Pad3)
- D13 pad 2: Net-(D13-Pad2) -> +5V
- D13 pad 3: GND -> Net-(D13-Pad3)
- D13 pad 4: Net-(D12-Pad2) -> GND
- D14 pad 1: +5V -> Net-(D12-Pad3)
- D14 pad 2: Net-(D14-Pad2) -> +5V
- D14 pad 3: GND -> Net-(D14-Pad3)
- D14 pad 4: Net-(D13-Pad2) -> GND
- D15 pad 1: +5V -> Net-(D14-Pad3)
- D15 pad 2: Net-(D15-Pad2) -> +5V
- D15 pad 3: GND -> Net-(D15-Pad3)
- D15 pad 4: Net-(D14-Pad2) -> GND
- D16 pad 1: +5V -> Net-(D15-Pad3)
- D16 pad 2: Net-(D16-Pad2) -> +5V
- D16 pad 3: GND -> Net-(D16-Pad3)
- D16 pad 4: Net-(D15-Pad2) -> GND
- D17 pad 1: +5V -> Net-(D15-Pad3)
- D17 pad 2: Net-(D17-Pad2) -> +5V
- D17 pad 3: GND -> Net-(D17-Pad3)
- D17 pad 4: Net-(D16-Pad2) -> GND
- D18 pad 1: +5V -> Net-(D17-Pad3)
- D18 pad 2: Net-(D18-Pad2) -> +5V
- D18 pad 3: GND -> Net-(D18-Pad3)
- D18 pad 4: Net-(D17-Pad2) -> GND
- D19 pad 1: +5V -> Net-(D18-Pad3)
- D19 pad 2: Net-(D19-Pad2) -> +5V
- D19 pad 3: GND -> Net-(D19-Pad3)
- D19 pad 4: Net-(D18-Pad2) -> GND
- D2 pad 1: +5V -> /RGB_DO_BUF
- D2 pad 2: Net-(D2-Pad2) -> +5V
- D2 pad 3: GND -> Net-(D2-Pad3)
- D2 pad 4: Net-(D1-Pad2) -> GND
- D20 pad 1: +5V -> Net-(D18-Pad3)
- D20 pad 2: Net-(D20-Pad2) -> +5V
- D20 pad 3: GND -> Net-(D20-Pad3)
- D20 pad 4: Net-(D19-Pad2) -> GND
- D21 pad 1: +5V -> Net-(D20-Pad3)
- D21 pad 2: Net-(D21-Pad2) -> +5V
- D21 pad 3: GND -> Net-(D21-Pad3)
- D21 pad 4: Net-(D20-Pad2) -> GND
- D22 pad 1: +5V -> Net-(D21-Pad3)
- D22 pad 2: Net-(D22-Pad2) -> +5V
- D22 pad 3: GND -> Net-(D22-Pad3)
- D22 pad 4: Net-(D21-Pad2) -> GND
- D23 pad 1: +5V -> Net-(D21-Pad3)
- D23 pad 2: Net-(D23-Pad2) -> +5V
- D23 pad 3: GND -> Net-(D23-Pad3)
- D23 pad 4: Net-(D22-Pad2) -> GND
- D24 pad 1: +5V -> Net-(D23-Pad3)
- D24 pad 2: Net-(D24-Pad2) -> +5V
- D24 pad 3: GND -> Net-(D24-Pad3)
- D24 pad 4: Net-(D23-Pad2) -> GND
- D25 pad 1: +5V -> Net-(D24-Pad3)
- D25 pad 2: Net-(D25-Pad2) -> +5V
- D25 pad 3: GND -> Net-(D25-Pad3)
- D25 pad 4: Net-(D24-Pad2) -> GND
- D26 pad 1: +5V -> Net-(D24-Pad3)
- D26 pad 2: Net-(D26-Pad2) -> +5V
- D26 pad 3: GND -> Net-(D26-Pad3)
- D26 pad 4: Net-(D25-Pad2) -> GND
- D27 pad 1: +5V -> Net-(D26-Pad3)
- D27 pad 2: Net-(D27-Pad2) -> +5V
- D27 pad 3: GND -> Net-(D27-Pad3)
- D27 pad 4: Net-(D26-Pad2) -> GND
- D28 pad 1: +5V -> Net-(D27-Pad3)
- D28 pad 2: Net-(D28-Pad2) -> +5V
- D28 pad 3: GND -> Net-(D28-Pad3)
- D28 pad 4: Net-(D27-Pad2) -> GND
- D29 pad 1: +5V -> Net-(D27-Pad3)
- D29 pad 2: Net-(D29-Pad2) -> +5V
- D29 pad 3: GND -> Net-(D29-Pad3)
- D29 pad 4: Net-(D28-Pad2) -> GND
- D3 pad 1: +5V -> Net-(D2-Pad3)
- D3 pad 2: Net-(D3-Pad2) -> +5V
- D3 pad 3: GND -> Net-(D3-Pad3)
- D3 pad 4: Net-(D2-Pad2) -> GND
- D30 pad 1: +5V -> Net-(D29-Pad3)
- D30 pad 2: Net-(D30-Pad2) -> +5V
- D30 pad 3: GND -> Net-(D30-Pad3)
- D30 pad 4: Net-(D29-Pad2) -> GND
- D31 pad 1: +5V -> Net-(D30-Pad3)
- D31 pad 2: Net-(D31-Pad2) -> +5V
- D31 pad 3: GND -> Net-(D31-Pad3)
- D31 pad 4: Net-(D30-Pad2) -> GND
- D4 pad 1: +5V -> Net-(D3-Pad3)
- D4 pad 2: Net-(D4-Pad2) -> +5V
- D4 pad 3: GND -> Net-(D4-Pad3)
- D4 pad 4: Net-(D3-Pad2) -> GND
- D5 pad 1: +5V -> Net-(D3-Pad3)
- D5 pad 2: Net-(D5-Pad2) -> +5V
- D5 pad 3: GND -> Net-(D5-Pad3)
- D5 pad 4: Net-(D4-Pad2) -> GND
- D6 pad 1: +5V -> Net-(D5-Pad3)
- D6 pad 2: Net-(D6-Pad2) -> +5V
- D6 pad 3: GND -> Net-(D6-Pad3)
- D6 pad 4: Net-(D5-Pad2) -> GND
- D7 pad 1: +5V -> Net-(D6-Pad3)
- D7 pad 2: Net-(D7-Pad2) -> +5V
- D7 pad 3: GND -> Net-(D7-Pad3)
- D7 pad 4: Net-(D6-Pad2) -> GND
- D8 pad 1: +5V -> Net-(D6-Pad3)
- D8 pad 2: Net-(D8-Pad2) -> +5V
- D8 pad 3: GND -> Net-(D8-Pad3)
- D8 pad 4: Net-(D7-Pad2) -> GND
- D9 pad 1: +5V -> Net-(D8-Pad3)
- D9 pad 2: Net-(D10-Pad4) -> +5V
- D9 pad 3: GND -> Net-(D10-Pad1)
- D9 pad 4: Net-(D8-Pad2) -> GND
- J3 pad 1: /SPARE_0 -> GND
- J3 pad 2: GND -> /AIR_LED_5
- J3 pad 3: /SPARE_1 -> /AIR_LED_3
- J3 pad 4: GND -> /AIR_LED_1
- J3 pad 5: /SPARE_2 -> /AIR_SENSOR_0
- J3 pad 6: GND -> /AIR_SENSOR_2
- J3 pad 7: /SPARE_3 -> /AIR_SENSOR_4
- J3 pad 8: GND -> +3V3
- J3 pad 9: /SPARE_4 -> +5V
- J4 pad 1: /LED_0_OUT -> /SPARE_4
- J4 pad 2: /LED_1_OUT -> GND
- J4 pad 3: /LED_2_OUT -> /SPARE_3
- J4 pad 4: Net-(J4-Pad4) -> GND
- J4 pad 5: VCC -> /SPARE_2
- J5 pad 1: +3V3 -> +5V
- J5 pad 2: GND -> /KEY_LED/DO
- J5 pad 3: /AIR_5 -> Net-(J5-Pad3)
- J5 pad 4: /AIR_2 -> GND
- U1 pad 10: /LED_0 -> /BARREL_DETECT
- U1 pad 11: /SPARE_3 -> /SPARE_0
- U1 pad 12: /SPARE_4 -> /SPARE_2
- U1 pad 13: /SPARE_5 -> /SPARE_1
- U1 pad 14: /SPARE_6 -> /AIR_LED_5
- U1 pad 19: /SPARE_1 -> /AIR_LED_3
- U1 pad 2: /TOUCH_3 -> /TOUCH_0
- U1 pad 20: /SPARE_0 -> /AIR_LED_1
- U1 pad 21: /SPARE_2 -> /AIR_LED_0
- U1 pad 22: /TOUCH_1 -> /AIR_LED_2
- U1 pad 23: /TOUCH_2 -> /AIR_LED_4
- U1 pad 25: /AIR_0 -> /AIR_SENSOR_0
- U1 pad 26: /AIR_3 -> /AIR_SENSOR_2
- U1 pad 27: /AIR_1 -> /AIR_SENSOR_4
- U1 pad 28: /AIR_4 -> /AIR_SENSOR_5
- U1 pad 29: /AIR_2 -> /AIR_SENSOR_3
- U1 pad 3: /TOUCH_0 -> /TOUCH_3
- U1 pad 30: /AIR_5 -> /AIR_SENSOR_1
- U1 pad 36: Net-(U1-Pad36) -> /SPARE_3
- U1 pad 37: Net-(U1-Pad37) -> /SPARE_4
- U1 pad 5: /MUX_1 -> /TOUCH_2
- U1 pad 6: /MUX_0 -> /TOUCH_1
- U1 pad 8: /LED_2 -> /MUX_1
- U1 pad 9: /LED_1 -> /MUX_0
Routing:
- net +5V: track 623.0 -> 1349.1 mm, vias 0 -> 3
- net GND: track 658.8 -> 1355.7 mm, vias 35 -> 43
- net /USB_D-: track 0.00 -> 609.8 mm, vias 0 -> 3
- net /USB_D+: track 0.00 -> 605.4 mm, vias 0 -> 4
- net /BARREL_DETECT: track 0.00 -> 593.4 mm, vias 0 -> 3
- net Net-(J5-Pad3): track 0.00 -> 539.5 mm
- net /AIR_2: track 480.1 -> 0.00 mm, vias 1 -> 0
- net /AIR_5: track 479.9 -> 0.00 mm, vias 1 -> 0
- net /AIR_1: track 474.2 -> 0.00 mm, vias 1 -> 0
- net /AIR_4: track 474.1 -> 0.00 mm, vias 1 -> 0
- net /AIR_0: track 468.4 -> 0.00 mm, vias 1 -> 0
- net /AIR_3: track 468.3 -> 0.00 mm, vias 1 -> 0
- net /SPARE_5: track 445.1 -> 0.00 mm
- net /SPARE_6: track 443.1 -> 0.00 mm
- net /AIR_LED_0: track 0.00 -> 257.9 mm
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Other:
- board size 480 x 160 mm -> 480 x 151 mm
- board text added: "+5V"
- board text added: "5V"
- board text added: "Barrel Jack"
- board text added: "D+"
- board text added: "D-"
- board text added: "DO"
- board text added: "Din"
- board text added: "Inner Pins"
- board text added: "L3"
- board text added: "L4"
- board text added: "L5"
- board text added: "Make sure to connect D+ and D- on the underside of the teensy before soldering!"
- board text added: "S0"
- board text added: "S1"
- board text added: "S2"
- board text added: "S3"
- board text added: "S4"
- board text added: "S5"
- board text added: "USB Breakout"
- board text added: "USB C"
- board text added: "Version FULL2.0"
- board text removed: "A0"
- board text removed: "A1"
- board text removed: "A2"
- board text removed: "A3"
- board text removed: "A4"
- board text removed: "A5"
- board text removed: "SP5"
- board text removed: "SP6"
- board text removed: "Teensy LC"
- board text removed: "VCC"
