File: PCB Files/Circuit-Teensy32-Full-Board/OpeNITHM-full.sch (KiCad schematic (older format))
At the start: 109 parts, among them J3 Conn_02x07_Odd_Even, J4 Conn_02x03_Odd_Even, J5 Conn_02x04_Odd_Even, U1 Teensy-LC, U2 74HC4051D, U3 74HC4051D, U4 74HC4051D, U5 74HC4051D

Commit message: Preliminary upload of the Fullboard v2.0 PCB, and it's separate LED board. Nothing here should be purchased, this is just uploaded for reviewing.
Parts:
- removed C10, C11, C12, C13, C14, C15, C16, C17, C18, C19, C20, C21, C22, C23, C24, C25, C26, C27, C28, C29, C30, C31, C32, C33, C34, C35, C5, C6, C7, C8, C9: 100nF, Capacitor_SMD:C_0603_1608Metric, symbol Device:C_Small
- removed D1, D10, D11, D12, D13, D14, D15, D16, D17, D18, D19, D2, D20, D21, D22, D23, D24, D25, D26, D27, D28, D29, D3, D30, D31, D4, D5, D6, D7, D8, D9: WS2812B-B, LED_SMD:LED_WS2812B_PLCC4_5.0x5.0mm_P3.2mm, symbol LED:WS2812B
- removed H17, H18: MountingHole, MountingHole:MountingHole_3.2mm_M3_ISO14580, symbol Mechanical:MountingHole
- removed J4: Conn_02x03_Odd_Even, Connector_PinHeader_2.54mm:PinHeader_2x03_P2.54mm_Horizontal, symbol Connector_Generic:Conn_02x03_Odd_Even
- removed J5: Conn_02x04_Odd_Even, Connector_PinHeader_2.54mm:PinHeader_2x04_P2.54mm_Horizontal, symbol Connector_Generic:Conn_02x04_Odd_Even
- removed JP1: SolderJumper_3_Open, Jumper:SolderJumper-3_P1.3mm_Open_RoundedPad1.0x1.5mm_NumberLabels, symbol Jumper:SolderJumper_3_Open
- removed R17, R18, R19: 33, Resistor_THT:R_Axial_DIN0207_L6.3mm_D2.5mm_P7.62mm_Horizontal, symbol Device:R
- removed R20, R21, R22, R23, R24, R25: R_AIR, Resistor_THT:R_Axial_DIN0204_L3.6mm_D1.6mm_P5.08mm_Horizontal, symbol Device:R
- added D48, D49: D_Schottky, Diode_SMD:D_SMA, symbol Device:D_Schottky
- added J1: USB_C_Receptacle, Connector_USB:USB_C_Receptacle_GCT_USB4085, symbol Connector:USB_C_Receptacle_USB2.0
- added J2, J3: Conn_01x09, Connector_JST:JST_PH_S9B-PH-K_1x09_P2.00mm_Horizontal, symbol Connector_Generic:Conn_01x09
- added J5, J6: Conn_01x04, Connector_JST:JST_PH_S4B-PH-K_1x04_P2.00mm_Horizontal, symbol Connector_Generic:Conn_01x04
- added J7: Barrel_Jack, Connector_BarrelJack:BarrelJack_Horizontal, symbol Connector:Barrel_Jack_Switch
- added J8: Conn_01x02, Connector_PinHeader_2.54mm:PinHeader_1x02_P2.54mm_Vertical, symbol Connector_Generic:Conn_01x02
- added LOGO3: Logo, OpeNITHM:openithm-logo, symbol Mechanical:Fiducial
- added R5, R6: 5.1k, Resistor_SMD:R_0603_1608Metric, symbol Device:R_Small_US
- added TP1: +5V, TestPoint:TestPoint_Pad_D1.5mm, symbol Connector:TestPoint
- added TP2: D-, TestPoint:TestPoint_Pad_D1.5mm, symbol Connector:TestPoint
- added TP3: D+, TestPoint:TestPoint_Pad_D1.5mm, symbol Connector:TestPoint
- added TP4: GND, TestPoint:TestPoint_Pad_D1.5mm, symbol Connector:TestPoint
- J4: renamed from J3; value Conn_02x07_Odd_Even -> Conn_02x05_Odd_Even; footprint Connector_PinHeader_2.54mm:PinHeader_2x07_P2.54mm_Horizontal -> Connector_PinHeader_2.54mm:PinHeader_2x05_P2.54mm_Horizontal; symbol Connector_Generic:Conn_02x07_Odd_Even -> Connector_Generic:Conn_02x05_Odd_Even
- LOGO2: footprint OpeNITHM:openithm-logo -> OpeNITHM:openithm-big
Connections:
- net LED_1 is gone; now on net MUX_0: U1.9 (7_RX3_MOSI0)
- net LED_2 is gone; now on net MUX_1: U1.8 (6_RX3_CS1_PWM)
- net +3V3: now also J2.8 (Pin_8), J3.8 (Pin_8)
- net +5V: now also D48.1 (K), D49.1 (K), J2.9 (Pin_9), J3.9 (Pin_9), J5.1 (Pin_1), J6.1 (Pin_1)
- net GND: now also J1.A1 (GND), J1.A12 (GND), J1.B1 (GND), J1.B12 (GND), J2.1 (Pin_1), J3.1 (Pin_1), J5.4 (Pin_4), J6.4 (Pin_4), J7.2, R5.1, R6.1, TP4.1; no longer J4.12 (Pin_12), J4.14 (Pin_14)
- net MUX_0: no longer U1.6 (4_TX1_PWM_Touch)
- net MUX_1: no longer U1.5 (3_RX1_PWM_Touch)
- net SPARE_0: now also J4.9 (Pin_9), U1.11 (9_RX2_PWM); no longer J4.1 (Pin_1), U1.20 (13_LED_SCK0)
- net SPARE_1: now also J4.7 (Pin_7), U1.13 (11_MOSI0); no longer J4.3 (Pin_3), U1.19 (26_A12/DAC)
- net SPARE_2: now also U1.12 (10_TX2_CS0_PWM); no longer U1.21 (14_A0_SCK0)
- net SPARE_3: now also J4.3 (Pin_3), U1.36 (24_A10); no longer J4.7 (Pin_7), U1.11 (9_RX2_PWM)
- net SPARE_4: now also J4.1 (Pin_1), U1.37 (25_A11); no longer J4.9 (Pin_9), U1.12 (10_TX2_CS0_PWM)
- net TOUCH_0: now also U1.2 (0_RX1_MOSI1_Touch); no longer U1.3 (1_TX1_MISO1_Touch)
- net TOUCH_1: now also U1.6 (4_TX1_PWM_Touch); no longer U1.22 (15_A1_Touch)
- net TOUCH_2: now also U1.5 (3_RX1_PWM_Touch); no longer U1.23 (16_A2_SCL0_PWM_Touch)
- net TOUCH_3: now also U1.3 (1_TX1_MISO1_Touch); no longer U1.2 (0_RX1_MOSI1_Touch)
- net USB_D+: now reaches U1.38 (D+)
- net USB_D+: now also J1.A6 (D+), J1.B6 (D+), J8.1 (Pin_1), TP3.1
- net USB_D-: now reaches U1.39 (D-)
- net USB_D-: now also J1.A7 (D-), J1.B7 (D-), J8.2 (Pin_2), TP2.1
- net AIR_0 renamed AIR_SENSOR_0
- net AIR_SENSOR_0: now also J3.5 (Pin_5)
- net AIR_1 renamed AIR_SENSOR_4
- net AIR_SENSOR_4: now also J3.7 (Pin_7)
- net AIR_2 renamed AIR_SENSOR_3
- net AIR_SENSOR_3: now also J2.3 (Pin_3)
- net AIR_3 renamed AIR_SENSOR_2
- net AIR_SENSOR_2: now also J3.6 (Pin_6)
- net AIR_4 renamed AIR_SENSOR_5
- net AIR_SENSOR_5: now also J2.2 (Pin_2)
- net AIR_5 renamed AIR_SENSOR_1
- net AIR_SENSOR_1: now also J2.4 (Pin_4)
- net LED_0 renamed BARREL_DETECT
- net BARREL_DETECT: now also J7.3
- removed net SPARE_5: J4.11 (Pin_11), U1.13 (11_MOSI0)
- net SPARE_6 renamed AIR_LED_5
- net AIR_LED_5: now also J3.2 (Pin_2); no longer J4.13 (Pin_13)
- new net: D48.2 (A), J1.A4 (VBUS), J1.A9 (VBUS), J1.B4 (VBUS), J1.B9 (VBUS), TP1.1
- new net: J1.A5 (CC1), R5.2
- new net: J1.B5 (CC2), R6.2
- new net: J5.3 (Pin_3), J6.2 (Pin_2)
- new net: D49.2 (A), J7.1
- new net AIR_LED_0: J2.5 (Pin_5), U1.21 (14_A0_SCK0)
- new net AIR_LED_1: J3.4 (Pin_4), U1.20 (13_LED_SCK0)
- new net AIR_LED_2: J2.6 (Pin_6), U1.22 (15_A1_Touch)
- new net AIR_LED_3: J3.3 (Pin_3), U1.19 (26_A12/DAC)
- new net AIR_LED_4: J2.7 (Pin_7), U1.23 (16_A2_SCL0_PWM_Touch)
- new net KEY_LED/DO: J5.2 (Pin_2)
Other:
- note added: "IR\nSensor\n #0"
- note added: "LED #0\n"
- note added: "LED #5\n"
- note added: "Left Air Board"
- note added: "Left Side Tower RGB Connector"
- note added: "Main Integrated Strip for Keys"
- note added: "Right Air Board"
- note added: "Right Side Tower RGB Connector"
- note added: "Teensy USB Connection Pads\n"
- note removed: "A"
- note removed: "A - Anode (Long Pin)\nK - Cathode (Short Pin, Flat Side)"
- note removed: "C"
- note removed: "Connected to off-board \nIR LEDs"
- note removed: "Connected to\n off-board\nphototransistors"
- note removed: "E"
- note removed: "IR LEDs"
- note removed: "IR Sensors"
- note removed: "IR\nSensor\n #6"
- note removed: "If using Phototransistor:\nC - Collector\nE - Emitter\n\nIf using Photodiode:\nC - Cathode (Short Pin, Flat Side)\nE - Anode (Long Pin)"
- note removed: "K"
- note removed: "LED #5"
- note removed: "LED #6"
- note removed: "NOTE:\nR_AIR is highly dependent on your \nIR leds and phototransistor/diodes.\nThey may range from \n10k Ohm to 2M Ohm."
- note removed: "To +3.3V"
- note removed: "Voltage Jumper"
- moved on the sheet: H1, H10, H11, H12, H13, H14, H15, H16, H2, H3, H4, H5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
