File: PCB Files/Circuit-Teensy32-Full-Board-side/OpeNITHM-full.kicad_pcb (KiCad board)
At the start: 2 copper layers, 480 x 151 mm, 143 parts, among them J1 USB_C_Receptacle, J2 Conn_01x09, J3 Conn_01x09, J4 Conn_02x05_Odd_Even, J5 Conn_01x04, J6 Conn_01x04, J7 Barrel_Jack, J8 Conn_01x02, U1 Teensy-LC, U2 74HC4051D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

Commit message: Minor trace edit. Has no impact on board function
Routing:
- net GND: vias 43 -> 42
