File: PCB Files/Addon-LED-Board/LEDBoard.sch (KiCad schematic (older format))
At the start: 96 parts, among them J1 Conn_01x03, J2 Conn_01x03

Commit message: Fixed addon LED board. Previous version will not work, pins were wrong
Parts:
- D1, D10, D11, D12, D13, D14, D15, D16, D17, D18, D19, D2, D20, D21, D22, D23, D24, D25, D26, D27, D28, D29, D3, D30, D31, D32, D33, D34, D35, D36, D37, D38, D39, D4, D40, D41, D42, D43, D44, D45, D46, D47, D5, D6, D7, D8, D9: symbol LED:SK6812_SIDE-A -> LED:WS2812B
Connections:
- net +5V: now also D1.1 (VDD), D10.1 (VDD), D11.1 (VDD), D12.1 (VDD), D13.1 (VDD), D14.1 (VDD), D15.1 (VDD), D16.1 (VDD), D17.1 (VDD), D18.1 (VDD), D19.1 (VDD), D2.1 (VDD), D20.1 (VDD), D21.1 (VDD), D22.1 (VDD), D23.1 (VDD), D24.1 (VDD), D25.1 (VDD), D26.1 (VDD), D27.1 (VDD), D28.1 (VDD), D29.1 (VDD), D3.1 (VDD), D30.1 (VDD), D31.1 (VDD), D32.1 (VDD), D33.1 (VDD), D34.1 (VDD), D35.1 (VDD), D36.1 (VDD), D37.1 (VDD), D38.1 (VDD), D39.1 (VDD), D4.1 (VDD), D40.1 (VDD), D41.1 (VDD), D42.1 (VDD), D43.1 (VDD), D44.1 (VDD), D45.1 (VDD), D46.1 (VDD), D47.1 (VDD), D5.1 (VDD), D6.1 (VDD), D7.1 (VDD), D8.1 (VDD), D9.1 (VDD); no longer D1.2 (VDD), D10.2 (VDD), D11.2 (VDD), D12.2 (VDD), D13.2 (VDD), D14.2 (VDD), D15.2 (VDD), D16.2 (VDD), D17.2 (VDD), D18.2 (VDD), D19.2 (VDD), D2.2 (VDD), D20.2 (VDD), D21.2 (VDD), D22.2 (VDD), D23.2 (VDD), D24.2 (VDD), D25.2 (VDD), D26.2 (VDD), D27.2 (VDD), D28.2 (VDD), D29.2 (VDD), D3.2 (VDD), D30.2 (VDD), D31.2 (VDD), D32.2 (VDD), D33.2 (VDD), D34.2 (VDD), D35.2 (VDD), D36.2 (VDD), D37.2 (VDD), D38.2 (VDD), D39.2 (VDD), D4.2 (VDD), D40.2 (VDD), D41.2 (VDD), D42.2 (VDD), D43.2 (VDD), D44.2 (VDD), D45.2 (VDD), D46.2 (VDD), D47.2 (VDD), D5.2 (VDD), D6.2 (VDD), D7.2 (VDD), D8.2 (VDD), D9.2 (VDD)
- net DI: now also D1.4 (DIN), D2.4 (DIN); no longer D1.1 (DIN), D2.1 (DIN)
- net DO: now also D47.2 (DOUT); no longer D47.3 (DOUT)
- net GND: now also D1.3 (VSS), D10.3 (VSS), D11.3 (VSS), D12.3 (VSS), D13.3 (VSS), D14.3 (VSS), D15.3 (VSS), D16.3 (VSS), D17.3 (VSS), D18.3 (VSS), D19.3 (VSS), D2.3 (VSS), D20.3 (VSS), D21.3 (VSS), D22.3 (VSS), D23.3 (VSS), D24.3 (VSS), D25.3 (VSS), D26.3 (VSS), D27.3 (VSS), D28.3 (VSS), D29.3 (VSS), D3.3 (VSS), D30.3 (VSS), D31.3 (VSS), D32.3 (VSS), D33.3 (VSS), D34.3 (VSS), D35.3 (VSS), D36.3 (VSS), D37.3 (VSS), D38.3 (VSS), D39.3 (VSS), D4.3 (VSS), D40.3 (VSS), D41.3 (VSS), D42.3 (VSS), D43.3 (VSS), D44.3 (VSS), D45.3 (VSS), D46.3 (VSS), D47.3 (VSS), D5.3 (VSS), D6.3 (VSS), D7.3 (VSS), D8.3 (VSS), D9.3 (VSS); no longer D1.4 (VSS), D10.4 (VSS), D11.4 (VSS), D12.4 (VSS), D13.4 (VSS), D14.4 (VSS), D15.4 (VSS), D16.4 (VSS), D17.4 (VSS), D18.4 (VSS), D19.4 (VSS), D2.4 (VSS), D20.4 (VSS), D21.4 (VSS), D22.4 (VSS), D23.4 (VSS), D24.4 (VSS), D25.4 (VSS), D26.4 (VSS), D27.4 (VSS), D28.4 (VSS), D29.4 (VSS), D3.4 (VSS), D30.4 (VSS), D31.4 (VSS), D32.4 (VSS), D33.4 (VSS), D34.4 (VSS), D35.4 (VSS), D36.4 (VSS), D37.4 (VSS), D38.4 (VSS), D39.4 (VSS), D4.4 (VSS), D40.4 (VSS), D41.4 (VSS), D42.4 (VSS), D43.4 (VSS), D44.4 (VSS), D45.4 (VSS), D46.4 (VSS), D47.4 (VSS), D5.4 (VSS), D6.4 (VSS), D7.4 (VSS), D8.4 (VSS), D9.4 (VSS)
- new net: D2.2 (DOUT), D3.4 (DIN)
- new net: D3.2 (DOUT), D4.4 (DIN), D5.4 (DIN)
- new net: D5.2 (DOUT), D6.4 (DIN)
- new net: D6.2 (DOUT), D7.4 (DIN), D8.4 (DIN)
- new net: D8.2 (DOUT), D9.4 (DIN)
- new net: D10.4 (DIN), D11.4 (DIN), D9.2 (DOUT)
- new net: D11.2 (DOUT), D12.4 (DIN)
- new net: D12.2 (DOUT), D13.4 (DIN), D14.4 (DIN)
- new net: D14.2 (DOUT), D15.4 (DIN)
- new net: D15.2 (DOUT), D16.4 (DIN), D17.4 (DIN)
- new net: D17.2 (DOUT), D18.4 (DIN)
- new net: D18.2 (DOUT), D19.4 (DIN), D20.4 (DIN)
- new net: D20.2 (DOUT), D21.4 (DIN)
- new net: D21.2 (DOUT), D22.4 (DIN), D23.4 (DIN)
- new net: D23.2 (DOUT), D24.4 (DIN)
- new net: D24.2 (DOUT), D25.4 (DIN), D26.4 (DIN)
- new net: D26.2 (DOUT), D27.4 (DIN)
- new net: D27.2 (DOUT), D28.4 (DIN), D29.4 (DIN)
- new net: D29.2 (DOUT), D30.4 (DIN)
- new net: D30.2 (DOUT), D31.4 (DIN), D32.4 (DIN)
- new net: D32.2 (DOUT), D33.4 (DIN)
- new net: D33.2 (DOUT), D34.4 (DIN), D35.4 (DIN)
- new net: D35.2 (DOUT), D36.4 (DIN)
- new net: D36.2 (DOUT), D37.4 (DIN), D38.4 (DIN)
- new net: D38.2 (DOUT), D39.4 (DIN)
- new net: D39.2 (DOUT), D40.4 (DIN), D41.4 (DIN)
- new net: D41.2 (DOUT), D42.4 (DIN)
- new net: D42.2 (DOUT), D43.4 (DIN), D44.4 (DIN)
- new net: D44.2 (DOUT), D45.4 (DIN)
- new net: D45.2 (DOUT), D46.4 (DIN), D47.4 (DIN)
Changed lines of the file:
@@
 Main Integrated Strip for Keys
 $Comp
-L LED:SK6812_SIDE-A D2
+L LED:WS2812B D2
 U 1 1 625EAA3A
 P 2400 2150
@@
 Connection ~ 3200 1850
 $Comp
-L LED:SK6812_SIDE-A D3
+L LED:WS2812B D3
 U 1 1 625EAA72
 P 3200 2150
@@
 Connection ~ 1600 1850
 $Comp
-L LED:SK6812_SIDE-A D1
+L LED:WS2812B D1
 U 1 1 625EAA41
 P 1600 2150
@@
 $EndComp
 $Comp
-L LED:SK6812_SIDE-A D5
+L LED:WS2812B D5
 U 1 1 632CF991
 P 4800 2150
@@
 Connection ~ 5600 1850
 $Comp
-L LED:SK6812_SIDE-A D6
+L LED:WS2812B D6
 U 1 1 632CF9AA
 P 5600 2150
@@
 Connection ~ 4000 1850
 $Comp
-L LED:SK6812_SIDE-A D4
+L LED:WS2812B D4
 U 1 1 632CF9B5
 P 4000 2150
@@
 $EndComp
 $Comp
-L LED:SK6812_SIDE-A D8
+L LED:WS2812B D8
 U 1 1 632D4510
 P 7200 2150
@@
 Connection ~ 8000 1850
 $Comp
-L LED:SK6812_SIDE-A D9
+L LED:WS2812B D9
 U 1 1 632D4529
 P 8000 2150
@@
 Connection ~ 6400 1850
 $Comp
-L LED:SK6812_SIDE-A D7
+L LED:WS2812B D7
 U 1 1 632D4534
 P 6400 2150
@@
 $EndComp
 $Comp
-L LED:SK6812_SIDE-A D11
+L LED:WS2812B D11
 U 1 1 632D8B81
 P 9600 2150
@@
 Connection ~ 10400 1850
 $Comp
-L LED:SK6812_SIDE-A D12
+L LED:WS2812B D12
 U 1 1 632D8B9A
 P 10400 2150
@@
 Connection ~ 8800 1850
 $Comp
-L LED:SK6812_SIDE-A D10
+L LED:WS2812B D10
 U 1 1 632D8BA5
 P 8800 2150
@@
 $EndComp
 $Comp
-L LED:SK6812_SIDE-A D14
+L LED:WS2812B D14
 U 1 1 6330B525
 P 9200 2850
@@
 Connection ~ 8400 3150
 $Comp
-L LED:SK6812_SIDE-A D15
+L LED:WS2812B D15
 U 1 1 6330B53E
 P 8400 2850
@@
 Connection ~ 10000 3150
 $Comp
-L LED:SK6812_SIDE-A D13
+L LED:WS2812B D13
 U 1 1 6330B549
 P 10000 2850
@@
 $EndComp
 $Comp
-L LED:SK6812_SIDE-A D17
+L LED:WS2812B D17
 U 1 1 6330B576
 P 6800 2850
@@
 Connection ~ 6000 3150
 $Comp
-L LED:SK6812_SIDE-A D18
+L LED:WS2812B D18
 U 1 1 6330B58F
 P 6000 2850
@@
 Connection ~ 7600 3150
 $Comp
-L LED:SK6812_SIDE-A D16
+L LED:WS2812B D16
 U 1 1 6330B59A
 P 7600 2850
@@
 $EndComp
 $Comp
-L LED:SK6812_SIDE-A D20
+L LED:WS2812B D20
 U 1 1 6330B5C3
 P 4400 2850
@@
 Connection ~ 3600 3150
 $Comp
-L LED:SK6812_SIDE-A D21
+L LED:WS2812B D21
 U 1 1 6330B5DC
 P 3600 2850
@@
 Connection ~ 5200 3150
 $Comp
-L LED:SK6812_SIDE-A D19
+L LED:WS2812B D19
 U 1 1 6330B5E7
 P 5200 2850
@@
 $EndComp
 $Comp
-L LED:SK6812_SIDE-A D23
+L LED:WS2812B D23
 U 1 1 6330B610
 P 2000 2850
@@
 Connection ~ 1200 3150
 $Comp
-L LED:SK6812_SIDE-A D24
+L LED:WS2812B D24
 U 1 1 6330B629
 P 1200 2850
@@
 Connection ~ 2800 3150
 $Comp
-L LED:SK6812_SIDE-A D22
+L LED:WS2812B D22
 U 1 1 6330B634
 P 2800 2850
@@
 $EndComp
 $Comp
-L LED:SK6812_SIDE-A D26
+L LED:WS2812B D26
 U 1 1 633BDB38
 P 2400 3550
@@
 Connection ~ 3200 3250
 $Comp
-L LED:SK6812_SIDE-A D27
+L LED:WS2812B D27
 U 1 1 633BDB51
 P 3200 3550
@@
 Connection ~ 1600 3250
 $Comp
-L LED:SK6812_SIDE-A D25
+L LED:WS2812B D25
 U 1 1 633BDB5C
 P 1600 3550
@@
 $EndComp
 $Comp
-L LED:SK6812_SIDE-A D29
+L LED:WS2812B D29
 U 1 1 633BDB89
 P 4800 3550
@@
 Connection ~ 5600 3250
 $Comp
-L LED:SK6812_SIDE-A D30
+L LED:WS2812B D30
 U 1 1 633BDBA2
 P 5600 3550
@@
 Connection ~ 4000 3250
 $Comp
-L LED:SK6812_SIDE-A D28
+L LED:WS2812B D28
 U 1 1 633BDBAD
 P 4000 3550
@@
 $EndComp
 $Comp
-L LED:SK6812_SIDE-A D32
+L LED:WS2812B D32
 U 1 1 633BDBD6
 P 7200 3550
@@
 Connection ~ 8000 3250
 $Comp
-L LED:SK6812_SIDE-A D33
+L LED:WS2812B D33
 U 1 1 633BDBEF
 P 8000 3550
@@
 Connection ~ 6400 3250
 $Comp
-L LED:SK6812_SIDE-A D31
+L LED:WS2812B D31
 U 1 1 633BDBFA
 P 6400 3550
@@
 $EndComp
 $Comp
-L LED:SK6812_SIDE-A D35
+L LED:WS2812B D35
 U 1 1 633BDC23
 P 9600 3550
@@
 Connection ~ 10400 3250
 $Comp
-L LED:SK6812_SIDE-A D36
+L LED:WS2812B D36
 U 1 1 633BDC3C
 P 10400 3550
@@
 Connection ~ 8800 3250
 $Comp
-L LED:SK6812_SIDE-A D34
+L LED:WS2812B D34
 U 1 1 633BDC47
 P 8800 3550
@@
 $EndComp
 $Comp
-L LED:SK6812_SIDE-A D38
+L LED:WS2812B D38
 U 1 1 633BDC70
 P 9200 4250
@@
 Connection ~ 8400 4550
 $Comp
-L LED:SK6812_SIDE-A D39
+L LED:WS2812B D39
 U 1 1 633BDC89
 P 8400 4250
@@
 Connection ~ 10000 4550
 $Comp
-L LED:SK6812_SIDE-A D37
+L LED:WS2812B D37
 U 1 1 633BDC94
 P 10000 4250
@@
 $EndComp
 $Comp
-L LED:SK6812_SIDE-A D41
+L LED:WS2812B D41
 U 1 1 633BDCBF
 P 6800 4250
@@
 Connection ~ 6000 4550
 $Comp
-L LED:SK6812_SIDE-A D42
+L LED:WS2812B D42
 U 1 1 633BDCD8
 P 6000 4250
@@
 Connection ~ 7600 4550
 $Comp
-L LED:SK6812_SIDE-A D40
+L LED:WS2812B D40
 U 1 1 633BDCE3
 P 7600 4250
@@
 $EndComp
 $Comp
-L LED:SK6812_SIDE-A D44
+L LED:WS2812B D44
 U 1 1 633BDD0C
 P 4400 4250
@@
 Connection ~ 3600 4550
 $Comp
-L LED:SK6812_SIDE-A D45
+L LED:WS2812B D45
 U 1 1 633BDD25
 P 3600 4250
@@
 Connection ~ 5200 4550
 $Comp
-L LED:SK6812_SIDE-A D43
+L LED:WS2812B D43
 U 1 1 633BDD30
 P 5200 4250
@@
 $EndComp
 $Comp
-L LED:SK6812_SIDE-A D47
+L LED:WS2812B D47
 U 1 1 633BDD59
 P 2000 4250
@@
 Connection ~ 2800 4550
 $Comp
-L LED:SK6812_SIDE-A D46
+L LED:WS2812B D46
 U 1 1 633BDD7D
 P 2800 4250
