File: PCB Files/Addon-LED-Board/LEDBoard_Panelize.kicad_pcb (KiCad board)
At the start: 2 copper layers, 458 x 19.9 mm, 224 parts, among them J1 Conn_01x03, J2 Conn_01x03

Commit message: Fixed addon LED board. Previous version will not work, pins were wrong
Parts:
- removed the REF** at (337.5, 76.6)
- removed the REF** at (85.5, 76.6)
- removed the REF** at (57.5, 76.6)
- removed the REF** at (29.5, 76.6)
- removed the REF** at (1.50, 76.6)
- removed the REF** at (-26.5, 76.6)
- removed the REF** at (-54.5, 76.6)
- removed the REF** at (309.5, 76.6)
- removed the REF** at (281.5, 76.6)
- removed the REF** at (-82.5, 76.6)
- removed the REF** at (253.5, 76.6)
- removed the REF** at (225.5, 76.6)
- removed the REF** at (197.5, 76.6)
- removed the REF** at (169.5, 76.6)
- removed the REF** at (141.5, 76.6)
- removed the REF** at (113.5, 76.6)
- added REF**: mousebite, mousebite:mousebite, F.Cu at (337.5, 76.5)
- added REF**: mousebite, mousebite:mousebite, F.Cu at (309.5, 76.5)
- added REF**: mousebite, mousebite:mousebite, F.Cu at (281.5, 76.5)
- added REF**: mousebite, mousebite:mousebite, F.Cu at (253.5, 76.5)
- added REF**: mousebite, mousebite:mousebite, F.Cu at (225.5, 76.5)
- added REF**: mousebite, mousebite:mousebite, F.Cu at (197.5, 76.5)
- added REF**: mousebite, mousebite:mousebite, F.Cu at (169.5, 76.5)
- added REF**: mousebite, mousebite:mousebite, F.Cu at (141.5, 76.5)
- added REF**: mousebite, mousebite:mousebite, F.Cu at (113.5, 76.5)
- added REF**: mousebite, mousebite:mousebite, F.Cu at (85.5, 76.5)
- added REF**: mousebite, mousebite:mousebite, F.Cu at (57.5, 76.5)
- added REF**: mousebite, mousebite:mousebite, F.Cu at (29.5, 76.5)
- added REF**: mousebite, mousebite:mousebite, F.Cu at (1.50, 76.5)
- added REF**: mousebite, mousebite:mousebite, F.Cu at (-26.5, 76.5)
- added REF**: mousebite, mousebite:mousebite, F.Cu at (-54.5, 76.5)
- added REF**: mousebite, mousebite:mousebite, F.Cu at (-82.5, 76.5)
- moved C12 9.33 mm to (272.3, 73.2)
- moved C6 9.33 mm to (328.3, 73.2)
- moved C9 9.33 mm to (300.3, 73.2)
- moved C14 9.33 mm to (253.7, 73.2)
- moved C16 9.33 mm to (235.0, 73.2)
- moved C17 9.33 mm to (225.7, 73.2)
- moved C19 9.33 mm to (207.0, 73.2)
- moved C20 9.33 mm to (197.7, 73.2)
- moved C22 9.33 mm to (179.0, 73.2)
- moved C23 9.33 mm to (169.7, 73.2)
- moved C25 9.33 mm to (151.0, 73.2)
- moved C26 9.33 mm to (141.7, 73.2)
- moved C28 9.33 mm to (123.0, 73.2)
- moved C30 9.33 mm to (104.3, 73.2)
- moved C33 9.33 mm to (76.3, 73.2)
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Connections:
- D1 pad 1: /DI -> +5V
- D1 pad 2: +5V -> Net-(D1-Pad2)
- D1 pad 3: Net-(D1-Pad3) -> GND
- D1 pad 4: GND -> /DI
- D10 pad 1: Net-(D10-Pad1) -> +5V
- D10 pad 2: +5V -> Net-(D10-Pad2)
- D10 pad 3: Net-(D10-Pad3) -> GND
- D10 pad 4: GND -> Net-(D10-Pad4)
- D11 pad 1: Net-(D10-Pad1) -> +5V
- D11 pad 2: +5V -> Net-(D11-Pad2)
- D11 pad 3: Net-(D11-Pad3) -> GND
- D11 pad 4: GND -> Net-(D10-Pad4)
- D12 pad 1: Net-(D11-Pad3) -> +5V
- D12 pad 2: +5V -> Net-(D12-Pad2)
- D12 pad 3: Net-(D12-Pad3) -> GND
- D12 pad 4: GND -> Net-(D11-Pad2)
- D13 pad 1: Net-(D12-Pad3) -> +5V
- D13 pad 2: +5V -> Net-(D13-Pad2)
- D13 pad 3: Net-(D13-Pad3) -> GND
- D13 pad 4: GND -> Net-(D12-Pad2)
- D14 pad 1: Net-(D12-Pad3) -> +5V
- D14 pad 2: +5V -> Net-(D14-Pad2)
- D14 pad 3: Net-(D14-Pad3) -> GND
- D14 pad 4: GND -> Net-(D12-Pad2)
- D15 pad 1: Net-(D14-Pad3) -> +5V
- D15 pad 2: +5V -> Net-(D15-Pad2)
- D15 pad 3: Net-(D15-Pad3) -> GND
- D15 pad 4: GND -> Net-(D14-Pad2)
- D16 pad 1: Net-(D15-Pad3) -> +5V
- D16 pad 2: +5V -> Net-(D16-Pad2)
- D16 pad 3: Net-(D16-Pad3) -> GND
- D16 pad 4: GND -> Net-(D15-Pad2)
- D17 pad 1: Net-(D15-Pad3) -> +5V
- D17 pad 2: +5V -> Net-(D17-Pad2)
- D17 pad 3: Net-(D17-Pad3) -> GND
- D17 pad 4: GND -> Net-(D15-Pad2)
- D18 pad 1: Net-(D17-Pad3) -> +5V
- D18 pad 2: +5V -> Net-(D18-Pad2)
- D18 pad 3: Net-(D18-Pad3) -> GND
- D18 pad 4: GND -> Net-(D17-Pad2)
- D19 pad 1: Net-(D18-Pad3) -> +5V
- D19 pad 2: +5V -> Net-(D19-Pad2)
- D19 pad 3: Net-(D19-Pad3) -> GND
- D19 pad 4: GND -> Net-(D18-Pad2)
- D2 pad 1: /DI -> +5V
- D2 pad 2: +5V -> Net-(D2-Pad2)
- D2 pad 3: Net-(D2-Pad3) -> GND
- D2 pad 4: GND -> /DI
- D20 pad 1: Net-(D18-Pad3) -> +5V
- D20 pad 2: +5V -> Net-(D20-Pad2)
- D20 pad 3: Net-(D20-Pad3) -> GND
- D20 pad 4: GND -> Net-(D18-Pad2)
- D21 pad 1: Net-(D20-Pad3) -> +5V
- D21 pad 2: +5V -> Net-(D21-Pad2)
- D21 pad 3: Net-(D21-Pad3) -> GND
- D21 pad 4: GND -> Net-(D20-Pad2)
- D22 pad 1: Net-(D21-Pad3) -> +5V
- D22 pad 2: +5V -> Net-(D22-Pad2)
- D22 pad 3: Net-(D22-Pad3) -> GND
- D22 pad 4: GND -> Net-(D21-Pad2)
- D23 pad 1: Net-(D21-Pad3) -> +5V
- D23 pad 2: +5V -> Net-(D23-Pad2)
- D23 pad 3: Net-(D23-Pad3) -> GND
- D23 pad 4: GND -> Net-(D21-Pad2)
- D24 pad 1: Net-(D23-Pad3) -> +5V
- D24 pad 2: +5V -> Net-(D24-Pad2)
- D24 pad 3: Net-(D24-Pad3) -> GND
- D24 pad 4: GND -> Net-(D23-Pad2)
- D25 pad 1: Net-(D24-Pad3) -> +5V
- D25 pad 2: +5V -> Net-(D25-Pad2)
- D25 pad 3: Net-(D25-Pad3) -> GND
- D25 pad 4: GND -> Net-(D24-Pad2)
- D26 pad 1: Net-(D24-Pad3) -> +5V
- D26 pad 2: +5V -> Net-(D26-Pad2)
- D26 pad 3: Net-(D26-Pad3) -> GND
- D26 pad 4: GND -> Net-(D24-Pad2)
- D27 pad 1: Net-(D26-Pad3) -> +5V
- D27 pad 2: +5V -> Net-(D27-Pad2)
- D27 pad 3: Net-(D27-Pad3) -> GND
- D27 pad 4: GND -> Net-(D26-Pad2)
- D28 pad 1: Net-(D27-Pad3) -> +5V
- D28 pad 2: +5V -> Net-(D28-Pad2)
- D28 pad 3: Net-(D28-Pad3) -> GND
- D28 pad 4: GND -> Net-(D27-Pad2)
- D29 pad 1: Net-(D27-Pad3) -> +5V
- D29 pad 2: +5V -> Net-(D29-Pad2)
- D29 pad 3: Net-(D29-Pad3) -> GND
- D29 pad 4: GND -> Net-(D27-Pad2)
- D3 pad 1: Net-(D2-Pad3) -> +5V
- D3 pad 2: +5V -> Net-(D3-Pad2)
- D3 pad 3: Net-(D3-Pad3) -> GND
- D3 pad 4: GND -> Net-(D2-Pad2)
- D30 pad 1: Net-(D29-Pad3) -> +5V
- D30 pad 2: +5V -> Net-(D30-Pad2)
- D30 pad 3: Net-(D30-Pad3) -> GND
- D30 pad 4: GND -> Net-(D29-Pad2)
- D31 pad 1: Net-(D30-Pad3) -> +5V
- D31 pad 2: +5V -> Net-(D31-Pad2)
- D31 pad 3: Net-(D31-Pad3) -> GND
- D31 pad 4: GND -> Net-(D30-Pad2)
- D32 pad 1: Net-(D30-Pad3) -> +5V
- D32 pad 2: +5V -> Net-(D32-Pad2)
- D32 pad 3: Net-(D32-Pad3) -> GND
- D32 pad 4: GND -> Net-(D30-Pad2)
- D33 pad 1: Net-(D32-Pad3) -> +5V
- D33 pad 2: +5V -> Net-(D33-Pad2)
- D33 pad 3: Net-(D33-Pad3) -> GND
- D33 pad 4: GND -> Net-(D32-Pad2)
- D34 pad 1: Net-(D33-Pad3) -> +5V
- D34 pad 2: +5V -> Net-(D34-Pad2)
- D34 pad 3: Net-(D34-Pad3) -> GND
- D34 pad 4: GND -> Net-(D33-Pad2)
- D35 pad 1: Net-(D33-Pad3) -> +5V
- D35 pad 2: +5V -> Net-(D35-Pad2)
- D35 pad 3: Net-(D35-Pad3) -> GND
- D35 pad 4: GND -> Net-(D33-Pad2)
- D36 pad 1: Net-(D35-Pad3) -> +5V
- D36 pad 2: +5V -> Net-(D36-Pad2)
- D36 pad 3: Net-(D36-Pad3) -> GND
- D36 pad 4: GND -> Net-(D35-Pad2)
- D37 pad 1: Net-(D36-Pad3) -> +5V
- D37 pad 2: +5V -> Net-(D37-Pad2)
- D37 pad 3: Net-(D37-Pad3) -> GND
- D37 pad 4: GND -> Net-(D36-Pad2)
- D38 pad 1: Net-(D36-Pad3) -> +5V
- D38 pad 2: +5V -> Net-(D38-Pad2)
- D38 pad 3: Net-(D38-Pad3) -> GND
- D38 pad 4: GND -> Net-(D36-Pad2)
- D39 pad 1: Net-(D38-Pad3) -> +5V
- D39 pad 2: +5V -> Net-(D39-Pad2)
- D39 pad 3: Net-(D39-Pad3) -> GND
- D39 pad 4: GND -> Net-(D38-Pad2)
- D4 pad 1: Net-(D3-Pad3) -> +5V
- D4 pad 2: +5V -> Net-(D4-Pad2)
- D4 pad 3: Net-(D4-Pad3) -> GND
- D4 pad 4: GND -> Net-(D3-Pad2)
- D40 pad 1: Net-(D39-Pad3) -> +5V
- D40 pad 2: +5V -> Net-(D40-Pad2)
- D40 pad 3: Net-(D40-Pad3) -> GND
- D40 pad 4: GND -> Net-(D39-Pad2)
- D41 pad 1: Net-(D39-Pad3) -> +5V
- D41 pad 2: +5V -> Net-(D41-Pad2)
- D41 pad 3: Net-(D41-Pad3) -> GND
- D41 pad 4: GND -> Net-(D39-Pad2)
- D42 pad 1: Net-(D41-Pad3) -> +5V
- D42 pad 2: +5V -> Net-(D42-Pad2)
- D42 pad 3: Net-(D42-Pad3) -> GND
- D42 pad 4: GND -> Net-(D41-Pad2)
- D43 pad 1: Net-(D42-Pad3) -> +5V
- D43 pad 2: +5V -> Net-(D43-Pad2)
- D43 pad 3: Net-(D43-Pad3) -> GND
- D43 pad 4: GND -> Net-(D42-Pad2)
- D44 pad 1: Net-(D42-Pad3) -> +5V
- D44 pad 2: +5V -> Net-(D44-Pad2)
- D44 pad 3: Net-(D44-Pad3) -> GND
- D44 pad 4: GND -> Net-(D42-Pad2)
- D45 pad 1: Net-(D44-Pad3) -> +5V
- D45 pad 2: +5V -> Net-(D45-Pad2)
- D45 pad 3: Net-(D45-Pad3) -> GND
- D45 pad 4: GND -> Net-(D44-Pad2)
- D46 pad 1: Net-(D45-Pad3) -> +5V
- D46 pad 2: +5V -> Net-(D46-Pad2)
- D46 pad 3: Net-(D46-Pad3) -> GND
- D46 pad 4: GND -> Net-(D45-Pad2)
- D47 pad 1: Net-(D45-Pad3) -> +5V
- D47 pad 2: +5V -> /DO
- D47 pad 3: /DO -> GND
- D47 pad 4: GND -> Net-(D45-Pad2)
- D5 pad 1: Net-(D3-Pad3) -> +5V
- D5 pad 2: +5V -> Net-(D5-Pad2)
- D5 pad 3: Net-(D5-Pad3) -> GND
- D5 pad 4: GND -> Net-(D3-Pad2)
- D6 pad 1: Net-(D5-Pad3) -> +5V
- D6 pad 2: +5V -> Net-(D6-Pad2)
- D6 pad 3: Net-(D6-Pad3) -> GND
- D6 pad 4: GND -> Net-(D5-Pad2)
- D7 pad 1: Net-(D6-Pad3) -> +5V
- D7 pad 2: +5V -> Net-(D7-Pad2)
- D7 pad 3: Net-(D7-Pad3) -> GND
- D7 pad 4: GND -> Net-(D6-Pad2)
- D8 pad 1: Net-(D6-Pad3) -> +5V
- D8 pad 2: +5V -> Net-(D8-Pad2)
- D8 pad 3: Net-(D8-Pad3) -> GND
- D8 pad 4: GND -> Net-(D6-Pad2)
- D9 pad 1: Net-(D8-Pad3) -> +5V
- D9 pad 2: +5V -> Net-(D10-Pad4)
- D9 pad 3: Net-(D10-Pad1) -> GND
- D9 pad 4: GND -> Net-(D8-Pad2)
Routing:
- net GND: track 593.1 -> 612.1 mm
- net Net-(D15-Pad3): track 18.5 -> 0.00 mm, vias 3 -> 0
- net Net-(D15-Pad2): track 0.00 -> 18.5 mm, vias 0 -> 3
- net Net-(D6-Pad3): track 18.5 -> 0.00 mm, vias 3 -> 0
- net Net-(D6-Pad2): track 0.00 -> 18.5 mm, vias 0 -> 3
- net Net-(D36-Pad3): track 18.5 -> 0.00 mm, vias 3 -> 0
- net Net-(D36-Pad2): track 0.00 -> 18.5 mm, vias 0 -> 3
- net Net-(D33-Pad3): track 18.5 -> 0.00 mm, vias 3 -> 0
- net Net-(D33-Pad2): track 0.00 -> 18.5 mm, vias 0 -> 3
- net Net-(D30-Pad3): track 18.5 -> 0.00 mm, vias 3 -> 0
- net Net-(D30-Pad2): track 0.00 -> 18.5 mm, vias 0 -> 3
- net Net-(D27-Pad3): track 18.5 -> 0.00 mm, vias 3 -> 0
- net Net-(D27-Pad2): track 0.00 -> 18.5 mm, vias 0 -> 3
- net Net-(D24-Pad3): track 18.5 -> 0.00 mm, vias 3 -> 0
- net Net-(D24-Pad2): track 0.00 -> 18.5 mm, vias 0 -> 3
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Other:
- board size 458 x 19.9 mm -> 458 x 20 mm
